Commit message: refactor(xleo_hand): simplify MJCF model with convex collision and proper wrist joints
- Replace CoACD decomposition OBJs with trimesh convex hull STLs for collision
- Merge 6 virtual wrist bodies into single body with multi-joint (MJCF native)
- Add default classes for visual/collision geom separation
- Configure wrist joints with damping, armature, and position actuators (kp/kv)
- Add motor actuators for all finger joints
- Update URDF collision meshes to use convex hulls
- Add export_convex_meshes.py script and models README
- Remove unused CoACD OBJ files and convex_hulls directory

File: mujoco_playground/_src/manipulation/xleo_hand/models/urdf/ftl_xleo.urdf (robot description, URDF)
Before this commit: robot xleo, 46 links, 45 joints
Links:
- link LINK_ARM_BASE_L: geometry collision mesh filename=../ftl_meshes/LINK_ARM_BASE_L.STL; visual mesh filename=../ftl_meshes/LINK_ARM_BASE_L.STL
- link LINK_ARM_BASE_R: geometry collision mesh filename=../ftl_meshes/LINK_ARM_BASE_R.STL; visual mesh filename=../ftl_meshes/LINK_ARM_BASE_R.STL
- link LINK_BASE: geometry collision mesh filename=../ftl_meshes/LINK_BASE.STL; visual mesh filename=../ftl_meshes/LINK_BASE.STL
- link LINK_ELBOW_L0: geometry collision mesh filename=../ftl_meshes/LINK_ELBOW_L0.STL; visual mesh filename=../ftl_meshes/LINK_ELBOW_L0.STL
- link LINK_ELBOW_L1: geometry collision mesh filename=../ftl_meshes/LINK_ELBOW_L1.STL; visual mesh filename=../ftl_meshes/LINK_ELBOW_L1.STL
- link LINK_ELBOW_R0: geometry collision mesh filename=../ftl_meshes/LINK_ELBOW_R0.STL; visual mesh filename=../ftl_meshes/LINK_ELBOW_R0.STL
- link LINK_ELBOW_R1: geometry collision mesh filename=../ftl_meshes/LINK_ELBOW_R1.STL; visual mesh filename=../ftl_meshes/LINK_ELBOW_R1.STL
- link LINK_F0_L0: geometry collision mesh filename=../ftl_meshes/LINK_F0_L0.STL; visual mesh filename=../ftl_meshes/LINK_F0_L0.STL
- link LINK_F0_L1: geometry collision mesh filename=../ftl_meshes/LINK_F0_L1.STL; visual mesh filename=../ftl_meshes/LINK_F0_L1.STL
- link LINK_F0_L2: geometry collision mesh filename=../ftl_meshes/LINK_F0_L2.STL; visual mesh filename=../ftl_meshes/LINK_F0_L2.STL
- link LINK_F0_R0: geometry collision mesh filename=../ftl_meshes/LINK_F0_L0.STL; visual mesh filename=../ftl_meshes/LINK_F0_L0.STL
- link LINK_F0_R1: geometry collision mesh filename=../ftl_meshes/LINK_F0_L1.STL; visual mesh filename=../ftl_meshes/LINK_F0_L1.STL
- link LINK_F0_R2: geometry collision mesh filename=../ftl_meshes/LINK_F0_L2.STL; visual mesh filename=../ftl_meshes/LINK_F0_L2.STL
- link LINK_F1_L0: geometry collision mesh filename=../ftl_meshes/LINK_F1_L0.STL; visual mesh filename=../ftl_meshes/LINK_F1_L0.STL
- link LINK_F1_L1: geometry collision mesh filename=../ftl_meshes/LINK_F1_L1.STL; visual mesh filename=../ftl_meshes/LINK_F1_L1.STL
- link LINK_F1_L2: geometry collision mesh filename=../ftl_meshes/LINK_F1_L2.STL; visual mesh filename=../ftl_meshes/LINK_F1_L2.STL
- link LINK_F1_R0: geometry collision mesh filename=../ftl_meshes/LINK_F1_L0.STL; visual mesh filename=../ftl_meshes/LINK_F1_L0.STL
- link LINK_F1_R1: geometry collision mesh filename=../ftl_meshes/LINK_F1_L1.STL; visual mesh filename=../ftl_meshes/LINK_F1_L1.STL
- link LINK_F1_R2: geometry collision mesh filename=../ftl_meshes/LINK_F1_L2.STL; visual mesh filename=../ftl_meshes/LINK_F1_L2.STL
- link LINK_F2_L0: geometry collision mesh filename=../ftl_meshes/LINK_F2_L0.STL; visual mesh filename=../ftl_meshes/LINK_F2_L0.STL
- link LINK_F2_L1: geometry collision mesh filename=../ftl_meshes/LINK_F2_L1.STL; visual mesh filename=../ftl_meshes/LINK_F2_L1.STL
- link LINK_F2_L2: geometry collision mesh filename=../ftl_meshes/LINK_F2_L2.STL; visual mesh filename=../ftl_meshes/LINK_F2_L2.STL
- link LINK_F2_R0: geometry collision mesh filename=../ftl_meshes/LINK_F2_L0.STL; visual mesh filename=../ftl_meshes/LINK_F2_L0.STL
- link LINK_F2_R1: geometry collision mesh filename=../ftl_meshes/LINK_F2_L1.STL; visual mesh filename=../ftl_meshes/LINK_F2_L1.STL
- link LINK_F2_R2: geometry collision mesh filename=../ftl_meshes/LINK_F2_L2.STL; visual mesh filename=../ftl_meshes/LINK_F2_L2.STL
- link LINK_HAND_BASE_L: geometry collision mesh filename=../ftl_meshes/LINK_HAND_BASE_L.STL; visual mesh filename=../ftl_meshes/LINK_HAND_BASE_L.STL
- link LINK_HAND_BASE_R: geometry collision mesh filename=../ftl_meshes/LINK_HAND_BASE_R.STL; visual mesh filename=../ftl_meshes/LINK_HAND_BASE_R.STL
- link LINK_NECK_M0: geometry collision mesh filename=../ftl_meshes/LINK_NECK_M0.STL; visual mesh filename=../ftl_meshes/LINK_NECK_M0.STL
- link LINK_NECK_M1: geometry collision mesh filename=../ftl_meshes/LINK_NECK_M1.STL; visual mesh filename=../ftl_meshes/LINK_NECK_M1.STL
- link LINK_SHOULDER_L0: geometry collision mesh filename=../ftl_meshes/LINK_SHOULDER_L0.STL; visual mesh filename=../ftl_meshes/LINK_SHOULDER_L0.STL
- link LINK_SHOULDER_L1: geometry collision mesh filename=../ftl_meshes/LINK_SHOULDER_L1.STL; visual mesh filename=../ftl_meshes/LINK_SHOULDER_L1.STL
- link LINK_SHOULDER_L2: geometry collision mesh filename=../ftl_meshes/LINK_SHOULDER_L2.STL; visual mesh filename=../ftl_meshes/LINK_SHOULDER_L2.STL
- link LINK_SHOULDER_R0: geometry collision mesh filename=../ftl_meshes/LINK_SHOULDER_R0.STL; visual mesh filename=../ftl_meshes/LINK_SHOULDER_R0.STL
- link LINK_SHOULDER_R1: geometry collision mesh filename=../ftl_meshes/LINK_SHOULDER_R1.STL; visual mesh filename=../ftl_meshes/LINK_SHOULDER_R1.STL
- link LINK_SHOULDER_R2: geometry collision mesh filename=../ftl_meshes/LINK_SHOULDER_R2.STL; visual mesh filename=../ftl_meshes/LINK_SHOULDER_R2.STL
- link LINK_WAIST_M0: geometry collision mesh filename=../ftl_meshes/LINK_WAIST_M0.STL; visual mesh filename=../ftl_meshes/LINK_WAIST_M0.STL
- link LINK_WAIST_M1: geometry collision mesh filename=../ftl_meshes/LINK_WAIST_M1.STL; visual mesh filename=../ftl_meshes/LINK_WAIST_M1.STL
- link LINK_WAIST_M2: geometry collision mesh filename=../ftl_meshes/LINK_WAIST_M2.STL; visual mesh filename=../ftl_meshes/LINK_WAIST_M2.STL
- link LINK_WAIST_M3: geometry collision mesh filename=../ftl_meshes/LINK_WAIST_M3.STL; visual mesh filename=../ftl_meshes/LINK_WAIST_M3.STL
- link LINK_WRIST_L0: geometry collision mesh filename=../ftl_meshes/LINK_WRIST_L0.STL; visual mesh filename=../ftl_meshes/LINK_WRIST_L0.STL
- link LINK_WRIST_L1: geometry collision mesh filename=../ftl_meshes/LINK_WRIST_L1.STL; visual mesh filename=../ftl_meshes/LINK_WRIST_L1.STL
- link LINK_WRIST_R0: geometry collision mesh filename=../ftl_meshes/LINK_WRIST_R0.STL; visual mesh filename=../ftl_meshes/LINK_WRIST_R0.STL
- link LINK_WRIST_R1: geometry collision mesh filename=../ftl_meshes/LINK_WRIST_R1.STL; visual mesh filename=../ftl_meshes/LINK_WRIST_R1.STL

File: mujoco_playground/_src/manipulation/xleo_hand/models/urdf/ftl_xleo_dual_hand.urdf (robot description, URDF)
Before this commit: robot xleo, 35 links, 34 joints
Links:
- link LINK_F0_L0: geometry collision mesh filename=../ftl_meshes/LINK_F0_L0_convex.stl; visual mesh filename=../ftl_meshes/LINK_F0_L0.STL
- link LINK_F0_L1: geometry collision mesh filename=../ftl_meshes/LINK_F0_L1_convex.stl; visual mesh filename=../ftl_meshes/LINK_F0_L1.STL
- link LINK_F0_L2: geometry collision mesh filename=../ftl_meshes/LINK_F0_L2_convex.stl; visual mesh filename=../ftl_meshes/LINK_F0_L2.STL
- link LINK_F0_R0: geometry collision mesh filename=../ftl_meshes/LINK_F0_L0_convex.stl; visual mesh filename=../ftl_meshes/LINK_F0_L0.STL
- link LINK_F0_R1: geometry collision mesh filename=../ftl_meshes/LINK_F0_L1_convex.stl; visual mesh filename=../ftl_meshes/LINK_F0_L1.STL
- link LINK_F0_R2: geometry collision mesh filename=../ftl_meshes/LINK_F0_L2_convex.stl; visual mesh filename=../ftl_meshes/LINK_F0_L2.STL
- link LINK_F1_L0: geometry collision mesh filename=../ftl_meshes/LINK_F1_L0_convex.stl; visual mesh filename=../ftl_meshes/LINK_F1_L0.STL
- link LINK_F1_L1: geometry collision mesh filename=../ftl_meshes/LINK_F1_L1_convex.stl; visual mesh filename=../ftl_meshes/LINK_F1_L1.STL
- link LINK_F1_L2: geometry collision mesh filename=../ftl_meshes/LINK_F1_L2_convex.stl; visual mesh filename=../ftl_meshes/LINK_F1_L2.STL
- link LINK_F1_R0: geometry collision mesh filename=../ftl_meshes/LINK_F1_L0_convex.stl; visual mesh filename=../ftl_meshes/LINK_F1_L0.STL
- link LINK_F1_R1: geometry collision mesh filename=../ftl_meshes/LINK_F1_L1_convex.stl; visual mesh filename=../ftl_meshes/LINK_F1_L1.STL
- link LINK_F1_R2: geometry collision mesh filename=../ftl_meshes/LINK_F1_L2_convex.stl; visual mesh filename=../ftl_meshes/LINK_F1_L2.STL
- link LINK_F2_L0: geometry collision mesh filename=../ftl_meshes/LINK_F2_L0_convex.stl; visual mesh filename=../ftl_meshes/LINK_F2_L0.STL
- link LINK_F2_L1: geometry collision mesh filename=../ftl_meshes/LINK_F2_L1_convex.stl; visual mesh filename=../ftl_meshes/LINK_F2_L1.STL
- link LINK_F2_L2: geometry collision mesh filename=../ftl_meshes/LINK_F2_L2_convex.stl; visual mesh filename=../ftl_meshes/LINK_F2_L2.STL
- link LINK_F2_R0: geometry collision mesh filename=../ftl_meshes/LINK_F2_L0_convex.stl; visual mesh filename=../ftl_meshes/LINK_F2_L0.STL
- link LINK_F2_R1: geometry collision mesh filename=../ftl_meshes/LINK_F2_L1_convex.stl; visual mesh filename=../ftl_meshes/LINK_F2_L1.STL
- link LINK_F2_R2: geometry collision mesh filename=../ftl_meshes/LINK_F2_L2_convex.stl; visual mesh filename=../ftl_meshes/LINK_F2_L2.STL
- link LINK_HAND_BASE_L: geometry collision mesh filename=../ftl_meshes/LINK_HAND_BASE_L_convex.stl; visual mesh filename=../ftl_meshes/LINK_HAND_BASE_L.STL
- link LINK_HAND_BASE_R: geometry collision mesh filename=../ftl_meshes/LINK_HAND_BASE_R_convex.stl; visual mesh filename=../ftl_meshes/LINK_HAND_BASE_R.STL
Joints:
- joint J_LINK_HAND_BASE_L_PITCH: limit lower=-3.14159 upper=3.14159 effort=5000 velocity=10 -> lower=-3.14159 upper=3.14159 effort=10 velocity=10
- joint J_LINK_HAND_BASE_L_ROLL: limit lower=-3.14159 upper=3.14159 effort=5000 velocity=10 -> lower=-3.14159 upper=3.14159 effort=10 velocity=10
- joint J_LINK_HAND_BASE_L_X: limit lower=-0.5 upper=0.5 effort=5000 velocity=10 -> lower=-0.5 upper=0.5 effort=10 velocity=10
- joint J_LINK_HAND_BASE_L_Y: limit lower=-0.5 upper=0.5 effort=5000 velocity=10 -> lower=-0.5 upper=0.5 effort=10 velocity=10
- joint J_LINK_HAND_BASE_L_YAW: limit lower=-3.14159 upper=3.14159 effort=5000 velocity=10 -> lower=-3.14159 upper=3.14159 effort=10 velocity=10
- joint J_LINK_HAND_BASE_L_Z: limit lower=-0.5 upper=0.5 effort=5000 velocity=10 -> lower=-0.5 upper=0.5 effort=10 velocity=10
- joint J_LINK_HAND_BASE_R_PITCH: limit lower=-3.14159 upper=3.14159 effort=5000 velocity=10 -> lower=-3.14159 upper=3.14159 effort=10 velocity=10
- joint J_LINK_HAND_BASE_R_ROLL: limit lower=-3.14159 upper=3.14159 effort=5000 velocity=10 -> lower=-3.14159 upper=3.14159 effort=10 velocity=10
- joint J_LINK_HAND_BASE_R_X: limit lower=-0.5 upper=0.5 effort=5000 velocity=10 -> lower=-0.5 upper=0.5 effort=10 velocity=10
- joint J_LINK_HAND_BASE_R_Y: limit lower=-0.5 upper=0.5 effort=5000 velocity=10 -> lower=-0.5 upper=0.5 effort=10 velocity=10
- joint J_LINK_HAND_BASE_R_YAW: limit lower=-3.14159 upper=3.14159 effort=5000 velocity=10 -> lower=-3.14159 upper=3.14159 effort=10 velocity=10
- joint J_LINK_HAND_BASE_R_Z: limit lower=-0.5 upper=0.5 effort=5000 velocity=10 -> lower=-0.5 upper=0.5 effort=10 velocity=10
