Commit message: feat(xleo_hand): 新增 massage2 环境并更新模型与数据工具
添加基于 DeepMimic 风格奖励的第二版按摩任务环境（50Hz 控制频率），
更新双手 URDF/XML 模型配置，重构 mink 数据生成和回放工具，
补充 50Hz 对比可视化图表。

File: mujoco_playground/_src/manipulation/xleo_hand/models/urdf/ftl_xleo_dual_hand.urdf (robot description, URDF)
Before this commit: robot xleo, 35 links, 34 joints
Joints:
- joint J_LINK_HAND_BASE_L_PITCH: limit lower=-3.14159 upper=3.14159 effort=10 velocity=10 -> lower=-3.14159 upper=3.14159 effort=30 velocity=10
- joint J_LINK_HAND_BASE_L_ROLL: limit lower=-3.14159 upper=3.14159 effort=10 velocity=10 -> lower=-3.14159 upper=3.14159 effort=30 velocity=10
- joint J_LINK_HAND_BASE_L_X: limit lower=-0.5 upper=0.5 effort=10 velocity=10 -> lower=-0.2 upper=0.2 effort=30 velocity=10
- joint J_LINK_HAND_BASE_L_Y: limit lower=-0.5 upper=0.5 effort=10 velocity=10 -> lower=-0.2 upper=0.2 effort=30 velocity=10
- joint J_LINK_HAND_BASE_L_YAW: limit lower=-3.14159 upper=3.14159 effort=10 velocity=10 -> lower=-3.14159 upper=3.14159 effort=30 velocity=10
- joint J_LINK_HAND_BASE_L_Z: limit lower=-0.5 upper=0.5 effort=10 velocity=10 -> lower=-0.2 upper=0.2 effort=30 velocity=10
- joint J_LINK_HAND_BASE_R_X: limit lower=-0.5 upper=0.5 effort=10 velocity=10 -> lower=-0.2 upper=0.2 effort=30 velocity=10
- joint J_LINK_HAND_BASE_R_Y: limit lower=-0.5 upper=0.5 effort=10 velocity=10 -> lower=-0.2 upper=0.2 effort=30 velocity=10
- joint J_LINK_HAND_BASE_R_Z: limit lower=-0.5 upper=0.5 effort=10 velocity=10 -> lower=-0.2 upper=0.2 effort=30 velocity=10
